File: prj-kicad/pmod-dac-ls.kicad_pcb (KiCad board)
At the start: 2 copper layers, 38.1 x 20.3 mm, 16 parts, among them J1 JUMPER, P1 PMOD, P2 CONN_3, Q1 BC846, Q2 BCP52T, U1 MCP4921, U2 MCP6001

Commit message: = ADD: Create production files for rev1
Parts:
- added C5: 10uF, pmod-dac-ls:SMD0805, F.Cu at (148.2, 99.8)
- added LOGO-OHW: VAL**, pmod-dac-ls:logo-ohw, F.Cu at (142.5, 111.0)
- added R6: 0, pmod-dac-ls:SMD0603, F.Cu at (145.0, 100.0)
- added agilack-11.5: 450px, pmod-dac-ls:logo-agilack-11.5, F.Cu at (138.8, 103.0)
- moved J1 0.75 mm to (143.8, 96.5)
Connections:
- U1 pad 6: +3.3V -> Net-(R6-Pad2)
Routing:
- net Net-(R6-Pad2): track 0.00 -> 4.21 mm
- net GND: track 76.8 -> 79.6 mm, vias 10 -> 11
- net +3.3V: track 60.1 -> 57.3 mm
